Commit message: Added a camera to robot model

File: src/my_robot/urdf/my_robot.xacro (robot description, xacro)
@@ -117,3 +117,33 @@
     </visual>
   </link>
+  <joint type="fixed" name="camera">
+    <origin xyz="0.2 0 0" rpy="0 0 0"/>
+    <child link="camera"/>
+    <parent link="chassis"/>
+    <axis xyz="0 1 0" rpy="0 0 0"/>
+  </joint>
+  <link name='camera'>
+    <inertial>
+      <mass value="0.1"/>
+      <origin xyz="0 0 0" rpy=" 0 0 0"/>
+      <inertia
+          ixx="1e-6" ixy="0" ixz="0"
+          iyy="1e-6" iyz="0"
+          izz="1e-6"
+      />
+      <box_inertia m="0.1" x="0.05" y="0.05" z="0.05"/>
+    </inertial>
+    <collision name='camera'>
+      <origin xyz="0 0 0" rpy=" 0 0 0"/>
+      <geometry>
+        <box size="0.05 0.05 0.05"/>
+      </geometry>
+    </collision>
+    <visual name='camera'>
+      <origin xyz="0 0 0" rpy=" 0 0 0"/>
+      <geometry>
+        <box size="0.05 0.05 0.05"/>
+      </geometry>
+    </visual>
+  </link>
 </robot>

Commit message: Added hokuyo lidar mesh and link to udrf file, changed color of wheels, chassis and camera

File: src/my_robot/urdf/my_robot.xacro (robot description, xacro)
@@ -2,4 +2,5 @@
 <robot name="my_robot" xmlns:xacro="http://www.ros.org/wiki/xacro">
   <link name="robot_footprint"></link>
+  <!-- CHASSIS -->
   <joint name="robot_footprint_joint" type="fixed">
     <origin xyz="0 0 0" rpy="0 0 0" />
@@ -55,4 +56,8 @@
     </visual>
   </link>
+  <gazebo reference="chassis">
+      <material>Gazebo/Blue</material>
+  </gazebo>
+  <!-- LEFT WHEEL -->
   <joint type="continuous" name="left_wheel_hinge">
     <origin xyz="0 0.15 0" rpy="0 0 0"/>
@@ -86,4 +91,8 @@
     </visual>
   </link>
+  <gazebo reference="left_wheel">
+      <material>Gazebo/Green</material>
+  </gazebo>
+  <!-- RIGHT WHEEL -->
   <joint type="continuous" name="right_wheel_hinge">
     <origin xyz="0 -0.15 0" rpy="0 0 0"/>
@@ -117,5 +126,9 @@
     </visual>
   </link>
-  <joint type="fixed" name="camera">
+  <gazebo reference="right_wheel">
+      <material>Gazebo/Green</material>
+  </gazebo>
+  <!-- CAMERA -->
+  <joint type="fixed" name="camera_joint">
     <origin xyz="0.2 0 0" rpy="0 0 0"/>
     <child link="camera"/>
@@ -134,5 +147,5 @@
       <box_inertia m="0.1" x="0.05" y="0.05" z="0.05"/>
     </inertial>
-    <collision name='camera'>
+    <collision name='camera_collision'>
       <origin xyz="0 0 0" rpy=" 0 0 0"/>
       <geometry>
@@ -140,5 +153,5 @@
       </geometry>
     </collision>
-    <visual name='camera'>
+    <visual name='camera_visual'>
       <origin xyz="0 0 0" rpy=" 0 0 0"/>
       <geometry>
@@ -147,3 +160,36 @@
     </visual>
   </link>
+  <gazebo reference="camera">
+      <material>Gazebo/Red</material>
+  </gazebo>
+  <!-- HOKUYO LIDAR -->
+  <joint type="fixed" name="hukoyo_joint">
+    <origin xyz="0.15 0 0.1" rpy="0 0 0"/>
+    <child link="hokuyo"/>
+    <parent link="chassis"/>
+    <axis xyz="0 1 0" rpy="0 0 0"/>
+  </joint>
+  <link name='hokuyo'>
+    <inertial>
+      <mass value="1e-5"/>
+      <origin xyz="0 0 0" rpy=" 0 0 0"/>
+      <inertia
+          ixx="1e-6" ixy="0" ixz="0"
+          iyy="1e-6" iyz="0"
+          izz="1e-6"
+      />
+    </inertial>
+    <collision name='hokuyo_collision'>
+      <origin xyz="0 0 0" rpy=" 0 0 0"/>
+      <geometry>
+        <box size="0.1 0.1 0.1"/>
+      </geometry>
+    </collision>
+    <visual name='hokuyo_visual'>
+      <origin xyz="0 0 0" rpy=" 0 0 0"/>
+      <geometry>
+        <mesh filename="package://my_robot/meshes/hokuyo.dae"/>
+      </geometry>
+    </visual>
+  </link>
 </robot>

Commit message: Fixed bug in my_robot.xacro file (angles of elements)

File: src/my_robot/urdf/my_robot.xacro (robot description, xacro)
@@ -72,5 +72,5 @@
     <inertial>
       <mass value="5.0"/>
-      <origin xyz="0.0 0 0" rpy=" 0 1.5707 0"/>
+      <origin xyz="0.0 0 0" rpy=" 0 1.5707 1.5707"/>
       <inertia
           ixx="0.1" ixy="0" ixz="0"
@@ -80,5 +80,5 @@
     </inertial>
     <collision name='left_wheel_collision'>
-      <origin xyz="0 0 0" rpy=" 0 1.5707 0"/>
+      <origin xyz="0 0 0" rpy=" 0 1.5707 1.5707"/>
       <geometry>
         <cylinder radius="0.1" length="0.05"/>
@@ -86,5 +86,5 @@
     </collision>
     <visual name='left_wheel_visual'>
-      <origin xyz="0 0 0" rpy=" 1.5707 0 0"/>
+      <origin xyz="0 0 0" rpy=" 0 1.5707 1.5707"/>
       <geometry>
         <cylinder radius="0.1" length="0.05"/>
@@ -107,5 +107,5 @@
     <inertial>
       <mass value="5.0"/>
-      <origin xyz="0.0 0 0" rpy=" 0 1.5707 0"/>
+      <origin xyz="0.0 0 0" rpy=" 0 1.5707 1.5707"/>
       <inertia
           ixx="0.1" ixy="0" ixz="0"
@@ -115,5 +115,5 @@
     </inertial>
     <collision name='right_wheel_collision'>
-      <origin xyz="0 0 0" rpy=" 0 1.5707 0"/>
+      <origin xyz="0 0 0" rpy=" 0 1.5707 1.5707"/>
       <geometry>
         <cylinder radius="0.1" length="0.05"/>
@@ -121,5 +121,5 @@
     </collision>
     <visual name='right_wheel_visual'>
-      <origin xyz="0 0 0" rpy=" 1.5707 0 0"/>
+      <origin xyz="0 0 0" rpy=" 0 1.5707 1.5707"/>
       <geometry>
         <cylinder radius="0.1" length="0.05"/>

Commit message: Changed my_world.world to oryginal (removed my_robot) and changed my_robot to cylinder-shaped

File: src/my_robot/urdf/my_robot.xacro (robot description, xacro)
@@ -10,5 +10,5 @@
   </joint>
   <link name='chassis'>
-    <pose>0 0 0.1 0 0 0</pose>
+    <pose>0 0 0.075 0 0 0</pose>
     <inertial>
       <mass value="15.0"/>
@@ -20,8 +20,8 @@
       />
     </inertial>
-    <collision name='collision'>
+    <collision name='chassis_collision'>
       <origin xyz="0 0 0" rpy=" 0 0 0"/>
       <geometry>
-        <box size=".4 .2 .1"/>
+        <cylinder radius=".15" length=".1"/>
       </geometry>
     </collision>
@@ -29,38 +29,38 @@
       <origin xyz="0 0 0" rpy=" 0 0 0"/>
       <geometry>
-        <box size=".4 .2 .1"/>
+        <cylinder radius=".15" length=".1"/>
       </geometry>
     </visual>
     <collision name='back_caster_collision'>
-      <origin xyz="-0.15 0 -0.05" rpy=" 0 0 0"/>
+      <origin xyz="-0.08 0 -0.05" rpy=" 0 0 0"/>
       <geometry>
-        <sphere radius="0.0499"/>
+        <sphere radius="0.02499"/>
       </geometry>
     </collision>
     <visual name='back_caster_visual'>
-      <origin xyz="-0.15 0 -0.05" rpy=" 0 0 0"/>
+      <origin xyz="-0.08 0 -0.05" rpy=" 0 0 0"/>
       <geometry>
-        <sphere radius="0.05"/>
+        <sphere radius="0.025"/>
       </geometry>
     </visual>
     <collision name='front_caster_collision'>
-      <origin xyz="0.15 0 -0.05" rpy=" 0 0 0"/>
+      <origin xyz="0.8 0 -0.05" rpy=" 0 0 0"/>
       <geometry>
-        <sphere radius="0.0499"/>
+        <sphere radius="0.02499"/>
       </geometry>
     </collision>
     <visual name='front_caster_visual'>
-      <origin xyz="0.15 0 -0.05" rpy=" 0 0 0"/>
+      <origin xyz="0.08 0 -0.05" rpy=" 0 0 0"/>
       <geometry>
-        <sphere radius="0.05"/>
+        <sphere radius="0.025"/>
       </geometry>
     </visual>
   </link>
   <gazebo reference="chassis">
-      <material>Gazebo/Blue</material>
+      <material>Gazebo/Red</material>
   </gazebo>
   <!-- LEFT WHEEL -->
   <joint type="continuous" name="left_wheel_hinge">
-    <origin xyz="0 0.15 0" rpy="0 0 0"/>
+    <origin xyz="0 0.175 -0.025" rpy="0 0 0"/>
     <child link="left_wheel"/>
     <parent link="chassis"/>
@@ -71,5 +71,5 @@
   <link name='left_wheel'>
     <inertial>
-      <mass value="5.0"/>
+      <mass value="1.0"/>
       <origin xyz="0.0 0 0" rpy=" 0 1.5707 1.5707"/>
       <inertia
@@ -82,5 +82,5 @@
       <origin xyz="0 0 0" rpy=" 0 1.5707 1.5707"/>
       <geometry>
-        <cylinder radius="0.1" length="0.05"/>
+        <cylinder radius="0.05" length="0.05"/>
       </geometry>
     </collision>
@@ -88,14 +88,14 @@
       <origin xyz="0 0 0" rpy=" 0 1.5707 1.5707"/>
       <geometry>
-        <cylinder radius="0.1" length="0.05"/>
+        <cylinder radius="0.05" length="0.05"/>
       </geometry>
     </visual>
   </link>
   <gazebo reference="left_wheel">
-      <material>Gazebo/Green</material>
+      <material>Gazebo/Black</material>
   </gazebo>
   <!-- RIGHT WHEEL -->
   <joint type="continuous" name="right_wheel_hinge">
-    <origin xyz="0 -0.15 0" rpy="0 0 0"/>
+    <origin xyz="0 -0.175 -0.025" rpy="0 0 0"/>
     <child link="right_wheel"/>
     <parent link="chassis"/>
@@ -106,5 +106,5 @@
   <link name='right_wheel'>
     <inertial>
-      <mass value="5.0"/>
+      <mass value="1.0"/>
       <origin xyz="0.0 0 0" rpy=" 0 1.5707 1.5707"/>
       <inertia
@@ -117,5 +117,5 @@
       <origin xyz="0 0 0" rpy=" 0 1.5707 1.5707"/>
       <geometry>
-        <cylinder radius="0.1" length="0.05"/>
+        <cylinder radius="0.05" length="0.05"/>
       </geometry>
     </collision>
@@ -123,14 +123,14 @@
       <origin xyz="0 0 0" rpy=" 0 1.5707 1.5707"/>
       <geometry>
-        <cylinder radius="0.1" length="0.05"/>
+        <cylinder radius="0.05" length="0.05"/>
       </geometry>
     </visual>
   </link>
   <gazebo reference="right_wheel">
-      <material>Gazebo/Green</material>
+      <material>Gazebo/Black</material>
   </gazebo>
   <!-- CAMERA -->
   <joint type="fixed" name="camera_joint">
-    <origin xyz="0.2 0 0" rpy="0 0 0"/>
+    <origin xyz="0.15 0 0" rpy="0 0 0"/>
     <child link="camera"/>
     <parent link="chassis"/>
@@ -162,9 +162,9 @@
   </link>
   <gazebo reference="camera">
-      <material>Gazebo/Red</material>
+      <material>Gazebo/Black</material>
   </gazebo>
   <!-- HOKUYO LIDAR -->
   <joint type="fixed" name="hukoyo_joint">
-    <origin xyz="0.15 0 0.1" rpy="0 0 0"/>
+    <origin xyz="0.125 0 0.085" rpy="0 0 0"/>
     <child link="hokuyo"/>
     <parent link="chassis"/>
